File: schematic/kicad_playground.sch (KiCad schematic (older format))
At the start: 5 parts

Commit message: Small update to schematic
The cache lib was added.
Connections:
- net labels added: +5V, GND
- wire segments 22 -> 23
- no-connect marks 0 -> 1
Changed lines of the file:
@@
 L Device:R R?
 U 1 1 5BC795B1
-P 4000 2200
-F 0 "R?" H 4070 2246 50  0000 L CNN
-F 1 "22K" H 4070 2155 50  0000 L CNN
-F 2 "" V 3930 2200 50  0001 C CNN
-F 3 "~" H 4000 2200 50  0001 C CNN
-	1    4000 2200
+P 4000 2350
+F 0 "R?" H 4070 2396 50  0000 L CNN
+F 1 "22K" H 4070 2305 50  0000 L CNN
+F 2 "" V 3930 2350 50  0001 C CNN
+F 3 "~" H 4000 2350 50  0001 C CNN
+	1    4000 2350
 	1    0    0    -1
 $EndComp
 Wire Wire Line
-	3550 2200 3550 2400
+	3550 2200 3550 2550
 Wire Wire Line
-	3550 2400 4000 2400
+	3550 2550 4000 2550
 Wire Wire Line
-	4000 2400 4000 2350
+	4000 2550 4000 2500
 Wire Wire Line
 	3550 2000 4000 2000
 Wire Wire Line
-	4000 2050 4000 2000
+	4000 2200 4000 2000
 Connection ~ 4000 2000
 Wire Wire Line
@@
 	4000 1000 4000 1600
 Connection ~ 3050 1000
-Wire Wire Line
-	3550 2550 3550 2400
-Connection ~ 3550 2400
+Connection ~ 3550 2550
 Wire Wire Line
 	3550 2550 3050 2550
@@
 $EndComp
 Wire Wire Line
-	3700 1450 3700 1500
+	3700 1400 3700 1500
 Wire Wire Line
-	3700 1050 3700 1000
+	3700 1100 3700 1000
 Connection ~ 3700 1000
 Wire Wire Line
 	3700 1000 4000 1000
+NoConn ~ 2550 2000
+$Comp
+L power:+5V #PWR?
+U 1 1 5BC7C18E
+P 2350 950
+F 0 "#PWR?" H 2350 800 50  0001 C CNN
+F 1 "+5V" H 2365 1123 50  0000 C CNN
+F 2 "" H 2350 950 50  0001 C CNN
+F 3 "" H 2350 950 50  0001 C CNN
+	1    2350 950
+	1    0    0    -1
+$EndComp
+Wire Wire Line
+	2350 950  2350 1000
+Connection ~ 2350 1000
+$Comp
+L power:GND #PWR?
+U 1 1 5BC7C401
+P 2450 2650
+F 0 "#PWR?" H 2450 2400 50  0001 C CNN
+F 1 "GND" H 2455 2477 50  0000 C CNN
+F 2 "" H 2450 2650 50  0001 C CNN
+F 3 "" H 2450 2650 50  0001 C CNN
+	1    2450 2650
+	1    0    0    -1
+$EndComp
+Wire Wire Line
+	2450 2650 2450 2550
+Connection ~ 2450 2550
 $EndSCHEMATC
